Commit message: Created LiDAR

File: description/gazebo_control.xacro (robot description, xacro)
@@ -25,10 +25,10 @@
         </plugin>
         <plugin filename="gz-sim-joint-state-publisher-system" name="gz::sim::systems::JointStatePublisher">
-        <!-- Force the topic to match the standard ROS topic -->
-        <topic>joint_states</topic>
-        <!-- List all the moving joints you want to track -->
-        <joint_name>base_left_wheel_joint</joint_name>
-        <joint_name>base_right_wheel_joint</joint_name>
-    </plugin>
+            <!-- Force the topic to match the standard ROS topic -->
+            <topic>joint_states</topic>
+            <!-- List all the moving joints you want to track -->
+            <joint_name>base_left_wheel_joint</joint_name>
+            <joint_name>base_right_wheel_joint</joint_name>
+        </plugin>
     </gazebo>
 </robot>

File: description/robot_core.xacro (robot description, xacro)
@@ -13,4 +13,7 @@
     <material name="black">
         <color rgba="0 0 0 1" />
+    </material>
+    <material name="red">
+        <color rgba="1 0 0 1" />
     </material>
     <!-- BASE LINK -->

Commit message: ros_gz_bridge & Front camera

File: description/gazebo_control.xacro (robot description, xacro)
@@ -3,18 +3,18 @@
     <gazebo>
         <plugin filename="gz-sim-diff-drive-system" name="gz::sim::systems::DiffDrive">
-            <!-- Wheel Joints -->
+            <!-- Wheel Information -->
             <left_joint>base_left_wheel_joint</left_joint>
             <right_joint>base_right_wheel_joint</right_joint>
-            <!-- Kinematics -->
             <wheel_separation>0.35</wheel_separation>
             <wheel_radius>0.05</wheel_radius>
+            <!-- Input -->
+            <topic>cmd_vel</topic>
             <!-- Limits -->
             <max_linear_acceleration>10.0</max_linear_acceleration>
-            <!-- Topic & TF Settings -->
-            <topic>cmd_vel</topic>
+            <!-- Output -->
             <odom_topic>odom</odom_topic>
             <frame_id>odom</frame_id>
             <child_frame_id>base_link</child_frame_id>
-            <odom_publisher_frequency>30</odom_publisher_frequency>
+            <odom_publish_frequency>30</odom_publish_frequency>
         </plugin>
         <plugin filename="gz-sim-pose-publisher-system" name="gz::sim::systems::PosePublisher">
@@ -25,10 +25,11 @@
         </plugin>
         <plugin filename="gz-sim-joint-state-publisher-system" name="gz::sim::systems::JointStatePublisher">
-            <!-- Force the topic to match the standard ROS topic -->
             <topic>joint_states</topic>
-            <!-- List all the moving joints you want to track -->
             <joint_name>base_left_wheel_joint</joint_name>
             <joint_name>base_right_wheel_joint</joint_name>
         </plugin>
+        <plugin filename="gz-sim-sensors-system" name="gz::sim::systems::Sensors">
+            <render_engine>ogre2</render_engine>
+        </plugin>
     </gazebo>
 </robot>

File: description/lidar.xacro (robot description, xacro)
@@ -1,5 +1,5 @@
 <?xml version="1.0"?>
 <robot xmlns:xacro="http://www.ros.org/wiki/xacro" >
-    <link name="lidar_frame">
+    <link name="laser_frame">
         <visual>
             <geometry>
@@ -17,19 +17,20 @@
         </xacro:inertial_cylinder>
     </link>
-    <joint name="lidar_joint" type="fixed">
+    <joint name="laser_joint" type="fixed">
         <parent link="chassis" />
-        <child link="lidar_frame" />
+        <child link="laser_frame" />
         <origin xyz="0.1 0 0.175" rpy="0 0 0" />
     </joint>
-    <gazebo reference="lidar_frame">
+    <gazebo reference="laser_joint">
+        <preserveFixedJoint>true</preserveFixedJoint>
+        <disableFixedJointLumping>true</disableFixedJointLumping>
+    </gazebo>
+    <gazebo reference="laser_frame">
         <material>Gazebo/Red</material>
-        <sensor name="laser" type="gpu_lidar">
+        <sensor name="gpu_lidar" type="gpu_lidar">
             <pose>0 0 0 0 0 0</pose>
-            <visualize>true</visualize>
+            <topic>scan</topic>
             <update_rate>10</update_rate>
-            <!-- Harmonic uses this topic tag to broadcast internally -->
-            <topic>scan</topic>
-            <!-- Force the frame ID so RViz knows where the data comes from -->
-            <gz_frame_id>lidar_frame</gz_frame_id>
+            <gz_frame_id>laser_frame</gz_frame_id>
             <lidar>
                 <scan>
@@ -44,5 +45,12 @@
                     <max>12</max>
                 </range>
+                <noise>
+                    <type>gaussian</type>
+                    <mean>0.0</mean>
+                    <stddev>0.001</stddev>
+                </noise>
             </lidar>
+            <always_on>1</always_on>
+            <visualize>1</visualize>
         </sensor>
     </gazebo>

File: description/robot_core.xacro (robot description, xacro)
@@ -26,5 +26,5 @@
                 <box size="0.4 0.3 0.15" />
             </geometry>
-            <origin xyz="0.15 0 0.075" />
+            <origin xyz="0.2 0 0.075" />
             <material name="white" />
         </visual>
