Commit message: Created visualization and physics

File: description/robot.urdf.xacro (robot description, xacro)
@@ -2,3 +2,4 @@
 <robot xmlns:xacro="http://www.ros.org/wiki/xacro"  name="robot">
     <xacro:include filename="robot_core.xacro" />
+    <xacro:include filename="gazebo_control.xacro" />
 </robot>

File: description/robot_core.xacro (robot description, xacro)
@@ -21,5 +21,5 @@
         <visual>
             <geometry>
-                <box size="0.3 0.3 0.15" />
+                <box size="0.4 0.3 0.15" />
             </geometry>
             <origin xyz="0.15 0 0.075" />
@@ -28,5 +28,5 @@
         <collision>
             <geometry>
-                <box size="0.3 0.3 0.15" />
+                <box size="0.4 0.3 0.15" />
             </geometry>
             <origin xyz="0.15 0 0.075" />
@@ -36,4 +36,7 @@
         </xacro:inertial_box>
     </link>
+    <gazebo reference="chassis">
+        <material>Gazebo/White</material>
+    </gazebo>
     <!-- LEFT WHEEL LINK -->
     <link name="left_wheel">
@@ -53,4 +56,7 @@
         </xacro:inertial_cylinder>
     </link>
+    <gazebo reference="left_wheel">
+        <material>Gazebo/Blue</material>
+    </gazebo>
     <!-- RIGHT WHEEL LINK -->
     <link name="right_wheel">
@@ -70,4 +76,7 @@
         </xacro:inertial_cylinder>
     </link>
+    <gazebo reference="right_wheel">
+        <material>Gazebo/Blue</material>
+    </gazebo>
     <!-- CASTER WHEEL LINK-->
     <link name="caster_wheel">
@@ -87,4 +96,9 @@
         </xacro:inertial_sphere>
     </link>
+    <gazebo reference="caster_wheel">
+        <material>Gazebo/Black</material>
+        <mu1 value="0.001"/>
+        <mu2 value="0.001"/>
+    </gazebo>
     <!-- CHASSIS JOINT -->
     <joint name="base_chassis_joint" type="fixed">
@@ -111,5 +125,5 @@
         <parent link="base_link" />
         <child link="caster_wheel" />
-        <origin xyz="0.12 0 0" />
+        <origin xyz="0.16 0 0" />
     </joint>
 </robot>

Commit message: add ros2_control

File: description/robot.urdf.xacro (robot description, xacro)
@@ -2,7 +2,8 @@
 <robot xmlns:xacro="http://www.ros.org/wiki/xacro"  name="robot">
     <xacro:include filename="robot_core.xacro" />
-    <xacro:include filename="gazebo_control.xacro" />
+    <!-- <xacro:include filename="gazebo_control.xacro" /> -->
+    <xacro:include filename="ros2_control.xacro" />
     <xacro:include filename="lidar.xacro" />
     <xacro:include filename="camera.xacro" />
-    <xacro:include filename="depth_camera.xacro" />
+    <!-- <xacro:include filename="depth_camera.xacro" /> -->
 </robot>

File: description/robot_core.xacro (robot description, xacro)
@@ -26,5 +26,5 @@
                 <box size="0.4 0.3 0.15" />
             </geometry>
-            <origin xyz="0.2 0 0.075" />
+            <origin xyz="0.15 0 0.075" />
             <material name="white" />
         </visual>
@@ -128,5 +128,5 @@
         <parent link="base_link" />
         <child link="caster_wheel" />
-        <origin xyz="0.16 0 0" />
+        <origin xyz="0.16 0 -0.05" />
     </joint>
 </robot>
