Commit message: Fixing Lidar bugs

File: description/lidar.xacro (robot description, xacro)
@@ -1,5 +1,5 @@
 <?xml version="1.0"?>
 <robot xmlns:xacro="http://www.ros.org/wiki/xacro" >
-    <link name="laser_frame">
+    <link name="lidar_link">
         <visual>
             <geometry>
@@ -17,14 +17,10 @@
         </xacro:inertial_cylinder>
     </link>
-    <joint name="laser_joint" type="fixed">
-        <parent link="chassis" />
-        <child link="laser_frame" />
+    <joint name="lidar_joint" type="fixed">
+        <parent link="base_link" />
+        <child link="lidar_link" />
         <origin xyz="0.1 0 0.175" rpy="0 0 0" />
     </joint>
-    <gazebo reference="laser_joint">
-        <preserveFixedJoint>true</preserveFixedJoint>
-        <disableFixedJointLumping>true</disableFixedJointLumping>
-    </gazebo>
-    <gazebo reference="laser_frame">
+    <gazebo reference="lidar_link">
         <material>Gazebo/Red</material>
         <sensor name="gpu_lidar" type="gpu_lidar">
@@ -32,5 +28,5 @@
             <topic>scan</topic>
             <update_rate>10</update_rate>
-            <gz_frame_id>laser_frame</gz_frame_id>
+            <gz_frame_id>lidar_link</gz_frame_id>
             <lidar>
                 <scan>

Commit message: Make teleop keyboard works with gazebo through ros control

File: description/lidar.xacro (robot description, xacro)
@@ -20,5 +20,5 @@
         <parent link="base_link" />
         <child link="lidar_link" />
-        <origin xyz="0.1 0 0.175" rpy="0 0 0" />
+        <origin xyz="0.1 0 0.25" rpy="0 0 0" />
     </joint>
     <gazebo reference="lidar_link">
